File: hardware/kicad/MagnetronController/MagnetronController.kicad_sch (KiCad schematic)
At the start: 2 parts, among them J7 Conn_02x05_Odd_Even, J8 Conn_02x13_Counter_Clockwise

Commit message: feat: break into multiple boards
Other:
- removed sheet Sensor Array
- removed sheet ui
- moved on the sheet: J8

Commit message: feat: updates
Parts:
- added H1, H2, H3, H4: MountingHole_Pad, MountingHole:MountingHole_3.2mm_M3_ISO7380_Pad_TopBottom, symbol Mechanical:MountingHole_Pad
Connections:
- net +5V: now also J8.22 (Pin_22)
- net GND: now also H1.1, H2.1, H3.1, H4.1
- net mcu/aux2_btn: no longer names the net of J8.17 (Pin_17)
Other:
- sheet mcu ports: added none; removed aux2_btn
