File: hardware/kicad/MagnetronController/mcu.kicad_sch (KiCad schematic)
At the start: 1 part, among them U10 Teensy4.1

Commit message: feat: updates
Connections:
- net aux2_btn is gone; now on net speed_encoder_btn: U10.29 (37_CS)
- net hall7: now also U10.18 (26_A12_MOSI1); no longer U10.37 (15_A1_RX3_SPDIF_IN)
- net speed_encoder_btn: no longer U10.18 (26_A12_MOSI1)
- no-connect marks 28 -> 29
