File: hardware/kicad/MagnetronController/MagnetronController.kicad_pcb (KiCad board)
At the start: 4 copper layers, 80 x 80 mm, 17 parts, among them J1 Conn_01x04, J10 Barrel_Jack, J2 DIN-5_180degree, J3 DIN-5_180degree, J7 Conn_02x05_Odd_Even, J8 Conn_02x13_Counter_Clockwise, SW9 SW_SPST, U10 Teensy4.1, U12 6N137

Commit message: feat: break into multiple boards
Routing:
- net Net-(A1-2A): track 20.4 -> 21.4 mm
- net Net-(A1-2B): track 21.0 -> 22.0 mm
- net GND: vias 1 -> 72
- added copper zone on B.Cu, net GND
- added copper zone on F.Cu, net GND
Other:
- board text added: "MIDI In"
- board text added: "MIDI Out"

Commit message: chore: cleanup
Routing:
- net GND: vias 72 -> 70
Changed lines of the file:
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@@
-	)
-	(via
-		(at 77.216 102.87)
-		(size 0.6)
-		(drill 0.3)
-		(layers "F.Cu" "B.Cu")
-		(free yes)
-		(net 2)
 	)
 	(via
@@
 	)
 	(via
-		(at 98.298 120.142)
-		(size 0.6)
-		(drill 0.3)
-		(layers "F.Cu" "B.Cu")
-		(free yes)
-		(net 2)
-	)
-	(via
 		(at 89.662 126.492)
 		(size 0.6)
@@
 	)
 	(via
-		(at 70.866 113.03)
-		(size 0.6)
-		(drill 0.3)
-		(layers "F.Cu" "B.Cu")
-		(free yes)
-		(net 2)
-	)
-	(via
-		(at 98.806 125.984)
-		(size 0.6)
-		(drill 0.3)
-		(layers "F.Cu" "B.Cu")
-		(free yes)
-		(net 2)
-	)
-	(via
-		(at 93.726 125.984)
+		(at 71.882 111.76)
+		(size 0.6)
+		(drill 0.3)
+		(layers "F.Cu" "B.Cu")
+		(free yes)
+		(net 2)
+	)
+	(via
+		(at 99.314 127)
+		(size 0.6)
+		(drill 0.3)
+		(layers "F.Cu" "B.Cu")
+		(free yes)
+		(net 2)
+	)
+	(via
+		(at 93.472 125.222)
 		(size 0.6)
 		(drill 0.3)
@@
 	)
 	(via
-		(at 61.722 91.44)
-		(size 0.6)
-		(drill 0.3)
+		(at 66.802 90.424)
+		(size 0.6)
+		(drill 0.3)

Commit message: feat: updates
Parts:
- removed J10: Barrel_Jack, Connector_BarrelJack:BarrelJack_CUI_PJ-102AH_Horizontal
- added C1: 100uf, Capacitor_THT:CP_Radial_D5.0mm_P2.50mm, F.Cu at (80.0, 101.3)
- added H1: MountingHole_Pad, MountingHole:MountingHole_3.2mm_M3_ISO7380_Pad_TopBottom, F.Cu at (55.4, 68.1)
- added H2: MountingHole_Pad, MountingHole:MountingHole_3.2mm_M3_ISO7380_Pad_TopBottom, F.Cu at (126.2, 68.1)
- added H3: MountingHole_Pad, MountingHole:MountingHole_3.2mm_M3_ISO7380_Pad_TopBottom, F.Cu at (55.4, 138.9)
- added H4: MountingHole_Pad, MountingHole:MountingHole_3.2mm_M3_ISO7380_Pad_TopBottom, F.Cu at (126.2, 138.9)
- added J4: Barrel_Jack_MountingPin, Connector_BarrelJack:BarrelJack_CUI_PJ-102AH_Horizontal, F.Cu at (108.5, 78.5)
- R4: value 470k -> 470
- moved A1 0.93 mm to (58.9, 98.3)
Connections:
- A1 pad 10: unconnected-(A1-MS1-Pad10) -> +3.3V
- A1 pad 11: unconnected-(A1-MS2-Pad11) -> +3.3V
- A1 pad 12: unconnected-(A1-MS3-Pad12) -> +3.3V
- J2 pad 2: unconnected-(J2-Pad2) -> GND
- J8 pad 17: /mcu/aux2_btn -> unconnected-(J8-Pin_17-Pad17)
- J8 pad 22: unconnected-(J8-Pin_22-Pad22) -> +5V
- U10 pad 18: /mcu/speed_encoder_btn -> /mcu/hall7
- U10 pad 29: /mcu/aux2_btn -> /mcu/speed_encoder_btn
- U10 pad 37: /mcu/hall7 -> unconnected-(U10-15_A1_RX3_SPDIF_IN-Pad37)
Routing:
- net +5V: track 87.3 -> 132.4 mm
- net /mcu/aux2_btn: track 43.2 -> 0.00 mm
- net /mcu/hall7: track 41.3 -> 67.2 mm
- net /mcu/speed_encoder_btn: track 20.6 -> 37.6 mm, vias 0 -> 1
- net +24V: track 78.5 -> 88.3 mm
- net /mcu/midi_tx: track 56.4 -> 58.0 mm
- net Net-(A1-1B): track 14.5 -> 15.4 mm
- net Net-(A1-1A): track 18.2 -> 19.2 mm
- net Net-(A1-2B): track 22.0 -> 22.9 mm
- net Net-(A1-2A): track 21.4 -> 22.3 mm
- net GND: vias 70 -> 66
Other:
- board text added: "A4988"

Commit message: chore: cleanup
Parts:
- pwr sw: renamed from SW9; value SW_SPST -> SW_SPST 24V
- moved pwr sw 18.1 mm to (103.6, 77.2)
- moved C9 9.89 mm to (92.6, 87.7), turned to 90 degrees
- moved R4 9.38 mm to (92.6, 94.7), turned to 90 degrees
- moved U12 8.36 mm to (82.5, 87.4), turned to 0 degrees
- moved J4 6.88 mm to (115.3, 77.9)
- moved C1 3.00 mm to (82.0, 99.1), turned to -90 degrees
Connections:
- J4 pad 1: +24V -> /power/VIN_SW_24V
- pwr sw pad 1: +24V -> /power/VIN_SW_24V
Routing:
- net +24V: track 88.3 -> 62.0 mm
- net /power/VIN_SW_24V: track 0.00 -> 12.0 mm
- net /mcu/midi_rx: track 38.0 -> 49.6 mm, vias 0 -> 1
- net +5V: track 132.4 -> 136.2 mm
- net /mcu/midi_tx: track 58.0 -> 55.6 mm
- net Net-(D1-A): track 26.8 -> 28.6 mm
- net GND: track 1.47 -> 0.00 mm, vias 66 -> 60
- net +3.3V: track 1.03 -> 1.57 mm

Commit message: chore: cleanup
Parts:
- added D2: SS34, Diode_SMD:D_SMA, F.Cu at (105.4, 78.0)
- added F1: Polyfuse, Fuse:Fuse_Bourns_MF-RHT300, F.Cu at (115.8, 81.8)
- C1: footprint Capacitor_THT:CP_Radial_D5.0mm_P2.50mm -> Capacitor_THT:CP_Radial_D8.0mm_P3.80mm
- R1: value 220 -> 10
- R2: value 220 -> 33
- SW9: renamed from pwr sw; footprint Connector_PinHeader_2.54mm:PinHeader_1x02_P2.54mm_Vertical -> Connector_JST:JST_XH_B2B-XH-AM_1x02_P2.50mm_Vertical
- moved SW9 9.43 mm to (101.3, 68.1)
- moved R2 6.27 mm to (97.5, 75.7), turned to 90 degrees
- moved C9 2.45 mm to (92.6, 85.3)
- moved U12 2.45 mm to (82.5, 84.9)
- moved R4 2.45 mm to (92.6, 92.2)
- moved C1 1.89 mm to (83.1, 97.5)
- moved A1 0.76 mm to (58.9, 97.5)
- moved J1 0.76 mm to (53.8, 88.1)
- moved J4 0.31 mm to (115.3, 77.6)
Connections:
- J4 pad 1: /power/VIN_SW_24V -> /power/VIN_FUSE_24V
- R2 pad 2: +5V -> +3.3V
- SW9 pad 1: /power/VIN_SW_24V -> +24V
- SW9 pad 2: +24V -> /power/DIODE_SW_24V
Routing:
- net /power/VIN_SW_24V: track 12.0 -> 0.00 mm
- net /power/DIODE_SW_24V: track 0.00 -> 8.55 mm
- net +24V: track 62.0 -> 69.8 mm
- net /power/FUSE_DIODE_24V: track 0.00 -> 5.57 mm
- net /power/VIN_FUSE_24V: track 0.00 -> 4.42 mm
- net +5V: track 136.2 -> 131.8 mm
- net /mcu/midi_rx: track 49.6 -> 52.1 mm
- net Net-(D1-K): track 22.5 -> 20.0 mm
- net Net-(D1-A): track 28.6 -> 27.0 mm
- net Net-(A1-2A): track 22.3 -> 20.7 mm
- net +3.3V: track 1.57 -> 3.09 mm, vias 1 -> 2
- net Net-(A1-2B): track 22.9 -> 23.8 mm
- net /mcu/stepper_step: track 40.5 -> 41.3 mm
- net /mcu/stepper_sleep: track 39.9 -> 40.7 mm
- net /mcu/stepper_dir: track 39.9 -> 40.7 mm
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Other:
- board text added: "pwr sw"
