File: hardware/kicad/MagnetronController/midi_audio.kicad_sch (KiCad schematic)
At the start: 9 parts, among them J2 DIN-5_180degree, J3 DIN-5_180degree, U12 6N137

Commit message: feat: updates
Parts:
- R4: value 470k -> 470
Connections:
- net GND: now also J2.2
- no-connect marks 5 -> 4
Changed lines of the file:
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@@
-	)
-	(no_connect
-		(at 60.325 60.96)
 	)
 	(no_connect
@@
 	(wire
 		(pts
-			(xy 71.755 68.58) (xy 74.295 68.58)
+			(xy 71.628 68.58) (xy 74.168 68.58)
 		)
 		(stroke
@@
 	(wire
 		(pts
-			(xy 55.245 53.34) (xy 64.135 53.34)
+			(xy 55.118 53.34) (xy 64.008 53.34)
 		)
 		(stroke
@@
 	(wire
 		(pts
-			(xy 55.245 68.58) (xy 64.135 68.58)
+			(xy 55.118 68.58) (xy 64.008 68.58)
 		)
 		(stroke
@@
 	(wire
 		(pts
-			(xy 71.755 53.34) (xy 78.105 53.34)
+			(xy 71.628 53.34) (xy 77.978 53.34)
+		)
+		(stroke
+			(width 0)
+			(type default)
+		)
+	)
+	(wire
+		(pts
+			(xy 60.198 60.96) (xy 62.484 60.96)
 		)
 		(stroke
@@
 	(hierarchical_label "midi_tx"
 		(shape input)
-		(at 74.295 68.58 0)
+		(at 74.168 68.58 0)
 		(effects
 			(font
@@
 			)
 			(justify left)
+		)
+	)
+	(symbol
+		(lib_id "power:GND")
+		(at 62.484 60.96 90)
+		(unit 1)
+		(exclude_from_sim no)
+		(in_bom yes)
+		(on_board yes)
+		(dnp no)
+		(property "Reference" "#PWR02"
+			(at 68.834 60.96 0)
+			(effects
+				(font
+					(size 1.27 1.27)
+				)
+				(hide yes)
+			)
+		)
+		(property "Value" "GND"
+			(at 66.294 60.9599 90)
+			(effects
+				(font
+					(size 1.27 1.27)
+				)
+				(justify right)
+			)
+		)
+		(property "Footprint" ""
+			(at 62.484 60.96 0)
+			(effects
+				(font
+					(size 1.27 1.27)
+				)
+				(hide yes)
+			)
+		)
+		(property "Datasheet" ""
+			(at 62.484 60.96 0)
+			(effects
+				(font
+					(size 1.27 1.27)
+				)
+				(hide yes)
+			)
+		)
+		(property "Description" "Power symbol creates a global label with name \"GND\" , ground"
+			(at 62.484 60.96 0)
+			(effects
+				(font
+					(size 1.27 1.27)
+				)
+				(hide yes)
+			)
+		)
+		(pin "1"
+		)
+		(instances
+			(project ""
+				(path "/a200339a-72b8-45b5-a453-e4d4f113bf3a/6fe42ffa-c8f4-41ce-934a-c3d504b77d4c"
+					(reference "#PWR02")
+					(unit 1)
+				)
+			)
 		)
 	)
@@
 			)
 		)
-		(property "Value" "470k"
+		(property "Value" "470"
 			(at 100.33 83.1849 0)
 			(effects
@@
 	(symbol
 		(lib_id "power:+5V")
-		(at 78.105 53.34 0)
+		(at 77.978 53.34 0)
 		(unit 1)
 		(exclude_from_sim no)
@@
 		(fields_autoplaced yes)
 		(property "Reference" "#PWR03"
-			(at 78.105 57.15 0)
+			(at 77.978 57.15 0)
 			(effects
 				(font
@@
 		)
 		(property "Value" "+5V"
-			(at 78.105 48.26 0)
+			(at 77.978 48.26 0)
 			(effects
 				(font
@@
 		)
 		(property "Footprint" ""
-			(at 78.105 53.34 0)
+			(at 77.978 53.34 0)
 			(effects
 				(font
@@
 		)
 		(property "Datasheet" ""
-			(at 78.105 53.34 0)
+			(at 77.978 53.34 0)
 			(effects
 				(font
@@
 		)
 		(property "Description" "Power symbol creates a global label with name \"+5V\""
-			(at 78.105 53.34 0)
+			(at 77.978 53.34 0)
 			(effects
 				(font
@@
 		(lib_name "DIN-5_180degree_1")
 		(lib_id "Connector:DIN-5_180degree")
-		(at 52.705 60.96 270)
+		(at 52.578 60.96 270)
 		(unit 1)
 		(exclude_from_sim no)
@@
 		(dnp no)
 		(property "Reference" "J2"
-			(at 53.34 60.96 90)
+			(at 53.213 60.96 90)
 			(effects
 				(font
@@
 		)
 		(property "Value" "DIN-5_180degree"
-			(at 60.96 55.245 90)
+			(at 60.833 55.245 90)
 			(effects
 				(font
@@
 		)
 		(property "Footprint" "music-table-footprints:MIDI_Wire_245"
-			(at 52.705 60.96 0)
+			(at 52.578 60.96 0)
 			(effects
 				(font
@@
 		)
 		(property "Datasheet" "http://www.mouser.com/ds/2/18/40_c091_abd_e-75918.pdf"
-			(at 52.705 60.96 0)
+			(at 52.578 60.96 0)
 			(effects
 				(font
@@
 		)
 		(property "Description" "5-pin DIN connector (5-pin DIN-5 stereo)"
-			(at 52.705 60.96 0)
+			(at 52.578 60.96 0)
 			(effects
 				(font
@@
 	(symbol
 		(lib_id "Device:R")
-		(at 67.945 53.34 90)
+		(at 67.818 53.34 90)
 		(unit 1)
 		(exclude_from_sim no)
@@
 		(dnp no)
 		(property "Reference" "R2"
-			(at 67.945 50.8 90)
+			(at 67.818 50.8 90)
 			(effects
 				(font
@@
 		)
 		(property "Value" "220"
-			(at 67.945 49.53 90)
+			(at 67.818 49.53 90)
 			(effects
 				(font
@@
 		)
 		(property "Footprint" "Resistor_SMD:R_0805_2012Metric_Pad1.20x1.40mm_HandSolder"
-			(at 67.945 55.118 90)
+			(at 67.818 55.118 90)
 			(effects
 				(font
@@
 		)
 		(property "Datasheet" "~"
-			(at 67.945 53.34 0)
+			(at 67.818 53.34 0)
 			(effects
 				(font
@@
 		)
 		(property "Description" "Resistor"
-			(at 67.945 53.34 0)
+			(at 67.818 53.34 0)
 			(effects
 				(font
@@
 	(symbol
 		(lib_id "Device:R")
-		(at 67.945 68.58 90)
+		(at 67.818 68.58 90)
 		(unit 1)
 		(exclude_from_sim no)
@@
 		(dnp no)
 		(property "Reference" "R1"
-			(at 67.945 66.04 90)
+			(at 67.818 66.04 90)
 			(effects
 				(font
@@
 		)
 		(property "Value" "220"
-			(at 67.945 64.77 90)
+			(at 67.818 64.77 90)
 			(effects
 				(font
@@
 		)
 		(property "Footprint" "Resistor_SMD:R_0805_2012Metric_Pad1.20x1.40mm_HandSolder"
-			(at 67.945 70.358 90)
+			(at 67.818 70.358 90)
 			(effects
 				(font
@@
 		)
 		(property "Datasheet" "~"
-			(at 67.945 68.58 0)
+			(at 67.818 68.58 0)
 			(effects
 				(font
@@
 		)
 		(property "Description" "Resistor"
-			(at 67.945 68.58 0)
-			(effects
-				(font
+			(at 67.818 68.58 0)
+			(effects
+				(font

Commit message: chore: cleanup
Parts:
- R1: value 220 -> 10
- R2: value 220 -> 33
Connections:
- net +3.3V: now also R2.2
- net +5V: no longer R2.2
Changed lines of the file:
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@@
-	)
-	(symbol
-		(lib_id "power:+5V")
-		(at 77.978 53.34 0)
-		(unit 1)
-		(exclude_from_sim no)
-		(in_bom yes)
-		(on_board yes)
-		(dnp no)
-		(fields_autoplaced yes)
-		(property "Reference" "#PWR03"
-			(at 77.978 57.15 0)
-			(effects
-				(font
-					(size 1.27 1.27)
-				)
-				(hide yes)
-			)
-		)
-		(property "Value" "+5V"
-			(at 77.978 48.26 0)
-			(effects
-				(font
-					(size 1.27 1.27)
-				)
-			)
-		)
-		(property "Footprint" ""
-			(at 77.978 53.34 0)
-			(effects
-				(font
-					(size 1.27 1.27)
-				)
-				(hide yes)
-			)
-		)
-		(property "Datasheet" ""
-			(at 77.978 53.34 0)
-			(effects
-				(font
-					(size 1.27 1.27)
-				)
-				(hide yes)
-			)
-		)
-		(property "Description" "Power symbol creates a global label with name \"+5V\""
-			(at 77.978 53.34 0)
-			(effects
-				(font
-					(size 1.27 1.27)
-				)
-				(hide yes)
-			)
-		)
-		(pin "1"
-		)
-		(instances
-			(project ""
-				(path "/a200339a-72b8-45b5-a453-e4d4f113bf3a/6fe42ffa-c8f4-41ce-934a-c3d504b77d4c"
-					(reference "#PWR03")
-					(unit 1)
-				)
-			)
-		)
 	)
 	(symbol
@@
 			)
 		)
-		(property "Value" "220"
-			(at 67.818 49.53 90)
-			(effects
-				(font
-					(size 1.27 1.27)
-				)
-				(hide yes)
+		(property "Value" "33"
+			(at 67.818 55.626 90)
+			(effects
+				(font
+					(size 1.27 1.27)
+				)
 			)
 		)
@@
 			)
 		)
-		(property "Value" "220"
-			(at 67.818 64.77 90)
-			(effects
-				(font
-					(size 1.27 1.27)
-				)
-				(hide yes)
+		(property "Value" "10"
+			(at 67.818 70.866 90)
+			(effects
+				(font
+					(size 1.27 1.27)
+				)
 			)
 		)
@@
 					(unit 1)
 				)
+			)
+		)
+	)
+	(symbol
+		(lib_id "power:+3.3V")
+		(at 77.978 53.34 0)
+		(unit 1)
+		(exclude_from_sim no)
+		(in_bom yes)
+		(on_board yes)
+		(dnp no)
+		(fields_autoplaced yes)
+		(property "Reference" "#PWR027"
+			(at 77.978 57.15 0)
+			(effects
+				(font
+					(size 1.27 1.27)
+				)
+				(hide yes)
+			)
+		)
+		(property "Value" "+3.3V"
+			(at 77.978 48.895 0)
+			(effects
+				(font
+					(size 1.27 1.27)
+				)
+			)
+		)
+		(property "Footprint" ""
+			(at 77.978 53.34 0)
+			(effects
+				(font
+					(size 1.27 1.27)
+				)
+				(hide yes)
+			)
+		)
+		(property "Datasheet" ""
+			(at 77.978 53.34 0)
+			(effects
+				(font
+					(size 1.27 1.27)
+				)
+				(hide yes)
+			)
+		)
+		(property "Description" "Power symbol creates a global label with name \"+3.3V\""
+			(at 77.978 53.34 0)
+			(effects
+				(font
+					(size 1.27 1.27)
+				)
+				(hide yes)
+			)
+		)
+		(pin "1"
+		)
+		(instances
+			(project "MagnetronController"
+				(path "/a200339a-72b8-45b5-a453-e4d4f113bf3a/6fe42ffa-c8f4-41ce-934a-c3d504b77d4c"
+					(reference "#PWR027")
+					(unit 1)
+				)
