File: hardware/kicad/MagnetronController/motor_driver.kicad_sch (KiCad schematic)
At the start: 2 parts, among them J1 Conn_01x04

Commit message: feat: updates
Parts:
- added C1: 100uf, Capacitor_THT:CP_Radial_D5.0mm_P2.50mm, symbol Device:C_Polarized
Connections:
- net +24V: now also C1.1
- net +3.3V: now also A1.10 (MS1), A1.11 (MS2), A1.12 (MS3)
- net GND: now also C1.2
- no-connect marks 3 -> 0
Changed lines of the file:
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@@
 	(paper "A4")
+	(junction
+		(at 92.71 91.44)
+		(diameter 0)
+		(color 0 0 0 0)
+	)
 	(junction
 		(at 102.87 63.5)
@@
 		(color 0 0 0 0)
 	)
-	(no_connect
-		(at 92.71 93.98)
-	)
-	(no_connect
-		(at 92.71 91.44)
-	)
-	(no_connect
-		(at 92.71 88.9)
-	)
-	(wire
-		(pts
-			(xy 107.95 58.42) (xy 107.95 63.5)
+	(junction
+		(at 107.95 58.928)
+		(diameter 0)
+		(color 0 0 0 0)
+	)
+	(junction
+		(at 90.678 71.12)
+		(diameter 0)
+		(color 0 0 0 0)
+	)
+	(wire
+		(pts
+			(xy 107.95 58.42) (xy 107.95 58.928)
 		)
 		(stroke
@@
 	(wire
 		(pts
+			(xy 90.678 71.12) (xy 92.71 71.12)
+		)
+		(stroke
+			(width 0)
+			(type default)
+		)
+	)
+	(wire
+		(pts
 			(xy 126.365 81.28) (xy 126.365 77.47)
 		)
@@
 	(wire
 		(pts
+			(xy 92.71 91.44) (xy 92.71 93.98)
+		)
+		(stroke
+			(width 0)
+			(type default)
+		)
+	)
+	(wire
+		(pts
+			(xy 92.71 88.9) (xy 92.71 91.44)
+		)
+		(stroke
+			(width 0)
+			(type default)
+		)
+	)
+	(wire
+		(pts
 			(xy 130.175 77.47) (xy 130.175 78.74)
 		)
@@
 	(wire
 		(pts
+			(xy 107.95 58.928) (xy 115.824 58.928)
+		)
+		(stroke
+			(width 0)
+			(type default)
+		)
+	)
+	(wire
+		(pts
+			(xy 107.95 58.928) (xy 107.95 63.5)
+		)
+		(stroke
+			(width 0)
+			(type default)
+		)
+	)
+	(wire
+		(pts
 			(xy 87.63 81.28) (xy 92.71 81.28)
 		)
@@
 	(wire
 		(pts
-			(xy 87.63 71.12) (xy 92.71 71.12)
+			(xy 87.63 71.12) (xy 90.678 71.12)
 		)
 		(stroke
@@
 		(pts
 			(xy 87.63 63.5) (xy 87.63 71.12)
+		)
+		(stroke
+			(width 0)
+			(type default)
+		)
+	)
+	(wire
+		(pts
+			(xy 92.71 91.44) (xy 90.678 91.44)
+		)
+		(stroke
+			(width 0)
+			(type default)
+		)
+	)
+	(wire
+		(pts
+			(xy 90.678 71.12) (xy 90.678 91.44)
 		)
 		(stroke
@@
 		(on_board yes)
 		(dnp no)
-		(fields_autoplaced yes)
 		(property "Reference" "A1"
 			(at 110.0933 60.96 0)
@@
 		)
 		(property "Value" "Pololu_Breakout_A4988"
-			(at 110.0933 63.5 0)
+			(at 114.3 71.374 0)
 			(effects
 				(font
@@
 					(unit 1)
 				)
+			)
+		)
+	)
+	(symbol
+		(lib_id "power:GND")
+		(at 123.444 58.928 90)
+		(unit 1)
+		(exclude_from_sim no)
+		(in_bom yes)
+		(on_board yes)
+		(dnp no)
+		(fields_autoplaced yes)
+		(property "Reference" "#PWR05"
+			(at 129.794 58.928 0)
+			(effects
+				(font
+					(size 1.27 1.27)
+				)
+				(hide yes)
+			)
+		)
+		(property "Value" "GND"
+			(at 127 58.9279 90)
+			(effects
+				(font
+					(size 1.27 1.27)
+				)
+				(justify right)
+			)
+		)
+		(property "Footprint" ""
+			(at 123.444 58.928 0)
+			(effects
+				(font
+					(size 1.27 1.27)
+				)
+				(hide yes)
+			)
+		)
+		(property "Datasheet" ""
+			(at 123.444 58.928 0)
+			(effects
+				(font
+					(size 1.27 1.27)
+				)
+				(hide yes)
+			)
+		)
+		(property "Description" "Power symbol creates a global label with name \"GND\" , ground"
+			(at 123.444 58.928 0)
+			(effects
+				(font
+					(size 1.27 1.27)
+				)
+				(hide yes)
+			)
+		)
+		(pin "1"
+		)
+		(instances
+			(project "MagnetronController"
+				(path "/a200339a-72b8-45b5-a453-e4d4f113bf3a/215a6cdd-134a-46bc-a137-d7b1ff5e8c97"
+					(reference "#PWR05")
+					(unit 1)
+				)
+			)
+		)
+	)
+	(symbol
+		(lib_id "Device:C_Polarized")
+		(at 119.634 58.928 90)
+		(unit 1)
+		(exclude_from_sim no)
+		(in_bom yes)
+		(on_board yes)
+		(dnp no)
+		(property "Reference" "C1"
+			(at 119.634 55.118 90)
+			(effects
+				(font
+					(size 1.27 1.27)
+				)
+			)
+		)
+		(property "Value" "100uf"
+			(at 118.745 54.61 90)
+			(effects
+				(font
+					(size 1.27 1.27)
+				)
+				(hide yes)
+			)
+		)
+		(property "Footprint" "Capacitor_THT:CP_Radial_D5.0mm_P2.50mm"
+			(at 123.444 57.9628 0)
+			(effects
+				(font
+					(size 1.27 1.27)
+				)
+				(hide yes)
+			)
+		)
+		(property "Datasheet" "~"
+			(at 119.634 58.928 0)
+			(effects
+				(font
+					(size 1.27 1.27)
+				)
+				(hide yes)
+			)
+		)
+		(property "Description" "Polarized capacitor"
+			(at 119.634 58.928 0)
+			(effects
+				(font
+					(size 1.27 1.27)
+				)
+				(hide yes)
+			)
+		)
+		(pin "1"
+		)
+		(pin "2"
+		)
+		(instances
+			(project ""
+				(path "/a200339a-72b8-45b5-a453-e4d4f113bf3a/215a6cdd-134a-46bc-a137-d7b1ff5e8c97"
+					(reference "C1")
+					(unit 1)
+				)

Commit message: chore: cleanup
Parts:
- C1: footprint Capacitor_THT:CP_Radial_D5.0mm_P2.50mm -> Capacitor_THT:CP_Radial_D8.0mm_P3.80mm
Changed lines of the file:
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@@
 			)
 		)
-		(property "Footprint" "Capacitor_THT:CP_Radial_D5.0mm_P2.50mm"
+		(property "Footprint" "Capacitor_THT:CP_Radial_D8.0mm_P3.80mm"
 			(at 123.444 57.9628 0)
 			(effects
