File: hardware/kicad/MagnetronController/power.kicad_sch (KiCad schematic)
At the start: 3 parts, among them J10 Barrel_Jack, SW9 SW_SPST

Commit message: feat: updates
Parts:
- removed J10: Barrel_Jack, Connector_BarrelJack:BarrelJack_CUI_PJ-102AH_Horizontal, symbol Connector:Barrel_Jack
- added J4: Barrel_Jack_MountingPin, Connector_BarrelJack:BarrelJack_CUI_PJ-102AH_Horizontal, symbol Connector:Barrel_Jack_MountingPin
Connections:
- net +24V: now also J4.1
- net GND: now also J4.2
Changed lines of the file:
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@@
+	)
+	(symbol
+		(lib_id "Connector:Barrel_Jack_MountingPin")
+		(at 46.99 73.66 0)
+		(unit 1)
+		(exclude_from_sim no)
+		(in_bom yes)
+		(on_board yes)
+		(dnp no)
+		(property "Reference" "J4"
+			(at 46.99 68.58 0)
+			(effects
+				(font
+					(size 1.27 1.27)
+				)
+			)
+		)
+		(property "Value" "Barrel_Jack_MountingPin"
+			(at 46.99 67.056 0)
+			(effects
+				(font
+					(size 1.27 1.27)
+				)
+				(hide yes)
+			)
+		)
+		(property "Footprint" "Connector_BarrelJack:BarrelJack_CUI_PJ-102AH_Horizontal"
+			(at 48.26 74.676 0)
+			(effects
+				(font
+					(size 1.27 1.27)
+				)
+				(hide yes)
+			)
+		)
+		(property "Datasheet" "~"
+			(at 48.26 74.676 0)
+			(effects
+				(font
+					(size 1.27 1.27)
+				)
+				(hide yes)
+			)
+		)
+		(property "Description" "DC Barrel Jack with a mounting pin"
+			(at 46.99 73.66 0)
+			(effects
+				(font
+					(size 1.27 1.27)
+				)
+				(hide yes)
+			)
+		)
+		(pin "2"
+		)
+		(pin "MP"
+		)
+		(pin "1"
+		)
+		(instances
+			(project ""
+				(path "/a200339a-72b8-45b5-a453-e4d4f113bf3a/1fa06de9-ef31-4bec-ac8d-485e9cffdee4"
+					(reference "J4")
+					(unit 1)
+				)
+			)
+		)
 	)
 	(symbol
@@
 					(unit 1)
 				)
-			)
-		)
-	)
-	(symbol
-		(lib_id "Connector:Barrel_Jack")
-		(at 46.99 73.66 0)
-		(unit 1)
-		(exclude_from_sim no)
-		(in_bom yes)
-		(on_board yes)
-		(dnp no)
-		(fields_autoplaced yes)
-		(property "Reference" "J10"
-			(at 46.99 65.405 0)
-			(effects
-				(font
-					(size 1.27 1.27)
-				)
-			)
-		)
-		(property "Value" "Barrel_Jack"
-			(at 46.99 67.945 0)
-			(effects
-				(font
-					(size 1.27 1.27)
-				)
-			)
-		)
-		(property "Footprint" "Connector_BarrelJack:BarrelJack_CUI_PJ-102AH_Horizontal"
-			(at 48.26 74.676 0)
-			(effects
-				(font
-					(size 1.27 1.27)
-				)
-				(hide yes)
-			)
-		)
-		(property "Datasheet" "~"
-			(at 48.26 74.676 0)
-			(effects
-				(font
-					(size 1.27 1.27)
-				)
-				(hide yes)
-			)
-		)
-		(property "Description" "DC Barrel Jack"
-			(at 46.99 73.66 0)
-			(effects
-				(font
-					(size 1.27 1.27)
-				)
-				(hide yes)
-			)
-		)
-		(pin "1"
-		)
-		(pin "2"
-		)
-		(instances
-			(project ""
-				(path "/a200339a-72b8-45b5-a453-e4d4f113bf3a/1fa06de9-ef31-4bec-ac8d-485e9cffdee4"
-					(reference "J10")
-					(unit 1)
-				)

Commit message: chore: cleanup
Parts:
- SW9: value SW_SPST -> SW_SPST 24V
Connections:
- net +24V: no longer J4.1, SW9.1 (A)
- new net VIN_SW_24V: J4.1, SW9.1 (A)
Changed lines of the file:
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@@
 	(paper "A4")
 	(junction
-		(at 49.784 61.214)
-		(diameter 0)
-		(color 0 0 0 0)
-	)
-	(junction
-		(at 58.42 61.214)
+		(at 68.58 61.468)
 		(diameter 0)
 		(color 0 0 0 0)
@@
 	(wire
 		(pts
-			(xy 58.42 59.69) (xy 58.42 61.214)
+			(xy 58.42 59.69) (xy 58.42 71.12)
 		)
 		(stroke
@@
 	(wire
 		(pts
+			(xy 68.58 61.468) (xy 68.58 71.12)
+		)
+		(stroke
+			(width 0)
+			(type default)
+		)
+	)
+	(wire
+		(pts
 			(xy 54.61 76.2) (xy 55.88 76.2)
 		)
@@
 	(wire
 		(pts
-			(xy 49.784 61.214) (xy 58.42 61.214)
-		)
-		(stroke
-			(width 0)
-			(type default)
-		)
-	)
-	(wire
-		(pts
 			(xy 54.61 71.12) (xy 58.42 71.12)
 		)
@@
 	(wire
 		(pts
-			(xy 68.58 59.69) (xy 68.58 71.12)
-		)
-		(stroke
-			(width 0)
-			(type default)
-		)
-	)
-	(wire
-		(pts
-			(xy 46.482 61.214) (xy 49.784 61.214)
-		)
-		(stroke
-			(width 0)
-			(type default)
-		)
-	)
-	(wire
-		(pts
-			(xy 58.42 61.214) (xy 58.42 71.12)
-		)
-		(stroke
-			(width 0)
-			(type default)
+			(xy 68.58 59.69) (xy 68.58 61.468)
+		)
+		(stroke
+			(width 0)
+			(type default)
+		)
+	)
+	(label "VIN_SW_24V"
+		(at 58.42 61.214 180)
+		(effects
+			(font
+				(size 1.27 1.27)
+			)
+			(justify right bottom)
 		)
 	)
@@
 	)
 	(symbol
-		(lib_id "power:+24V")
-		(at 46.482 61.214 90)
-		(unit 1)
-		(exclude_from_sim no)
-		(in_bom yes)
-		(on_board yes)
-		(dnp no)
-		(fields_autoplaced yes)
-		(property "Reference" "#PWR027"
-			(at 50.292 61.214 0)
-			(effects
-				(font
-					(size 1.27 1.27)
-				)
-				(hide yes)
-			)
-		)
-		(property "Value" "+24V"
-			(at 42.926 61.2139 90)
-			(effects
-				(font
-					(size 1.27 1.27)
-				)
-				(justify left)
-			)
-		)
-		(property "Footprint" ""
-			(at 46.482 61.214 0)
-			(effects
-				(font
-					(size 1.27 1.27)
-				)
-				(hide yes)
-			)
-		)
-		(property "Datasheet" ""
-			(at 46.482 61.214 0)
-			(effects
-				(font
-					(size 1.27 1.27)
-				)
-				(hide yes)
-			)
-		)
-		(property "Description" "Power symbol creates a global label with name \"+24V\""
-			(at 46.482 61.214 0)
-			(effects
-				(font
-					(size 1.27 1.27)
-				)
-				(hide yes)
-			)
-		)
-		(pin "1"
-		)
-		(instances
-			(project "Music Table"
-				(path "/a200339a-72b8-45b5-a453-e4d4f113bf3a/1fa06de9-ef31-4bec-ac8d-485e9cffdee4"
-					(reference "#PWR027")
-					(unit 1)
-				)
-			)
-		)
-	)
-	(symbol
 		(lib_id "Connector:Barrel_Jack_MountingPin")
 		(at 46.99 73.66 0)
@@
 		(on_board yes)
 		(dnp no)
-		(fields_autoplaced yes)
 		(property "Reference" "SW9"
-			(at 63.5 53.34 0)
-			(effects
-				(font
-					(size 1.27 1.27)
-				)
-			)
-		)
-		(property "Value" "SW_SPST"
+			(at 63.5 56.134 0)
+			(effects
+				(font
+					(size 1.27 1.27)
+				)
+			)
+		)
+		(property "Value" "SW_SPST 24V"
 			(at 63.5 55.88 0)
 			(effects
@@
 					(size 1.27 1.27)
 				)
+				(hide yes)
 			)
 		)
@@
 	(symbol
 		(lib_id "power:PWR_FLAG")
-		(at 49.784 61.214 0)
+		(at 68.58 61.468 270)
 		(unit 1)
 		(exclude_from_sim no)
@@
 		(fields_autoplaced yes)
 		(property "Reference" "#FLG02"
-			(at 49.784 59.309 0)
+			(at 70.485 61.468 0)
 			(effects
 				(font
@@
 		)
 		(property "Value" "PWR_FLAG"
-			(at 49.784 56.896 0)
-			(effects
-				(font
-					(size 1.27 1.27)
-				)
+			(at 72.644 61.4679 90)
+			(effects
+				(font
+					(size 1.27 1.27)
+				)
+				(justify left)
 			)
 		)
 		(property "Footprint" ""
-			(at 49.784 61.214 0)
+			(at 68.58 61.468 0)
 			(effects
 				(font
@@
 		)
 		(property "Datasheet" "~"
-			(at 49.784 61.214 0)
+			(at 68.58 61.468 0)
 			(effects
 				(font
@@
 		)
 		(property "Description" "Special symbol for telling ERC where power comes from"
-			(at 49.784 61.214 0)
-			(effects
-				(font
+			(at 68.58 61.468 0)
+			(effects
+				(font

Commit message: chore: cleanup
Parts:
- added D2: SS34, Diode_SMD:D_SMA, symbol Diode:SS34
- added F1: Polyfuse, Fuse:Fuse_Bourns_MF-RHT300, symbol Device:Polyfuse
- SW9: footprint Connector_PinHeader_2.54mm:PinHeader_1x02_P2.54mm_Vertical -> Connector_JST:JST_XH_B2B-XH-AM_1x02_P2.50mm_Vertical
Connections:
- net +24V: now also SW9.1 (A); no longer SW9.2 (B)
- net VIN_SW_24V renamed VIN_FUSE_24V
- net VIN_FUSE_24V: now also F1.1; no longer SW9.1 (A)
- new net DIODE_SW_24V: D2.1 (K), SW9.2 (B)
- new net FUSE_DIODE_24V: D2.2 (A), F1.2
Other:
- moved on the sheet: J4, SW9, U9
