File: hardware/kicad/MagnetronSensorArm/MagnetronSensorArm.kicad_sch (KiCad schematic)
At the start: 33 parts, among them J1 Conn_02x05_Odd_Even, U1 A1301KLHLT-T, U2 A1301KLHLT-T, U3 A1301KLHLT-T, U4 A1301KLHLT-T, U5 A1301KLHLT-T, U6 A1301KLHLT-T, U7 A1301KLHLT-T, U8 A1301KLHLT-T

Commit message: feat: cleanup
Parts:
- added H1: MountingHole_Pad, MountingHole:MountingHole_3.2mm_M3_ISO7380_Pad_TopBottom, symbol Mechanical:MountingHole_Pad
Connections:
- net GND: now also H1.1
Changed lines of the file:
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@@
 	(wire
 		(pts
+			(xy 87.63 40.64) (xy 87.63 43.434)
+		)
+		(stroke
+			(width 0)
+			(type default)
+		)
+	)
+	(wire
+		(pts
 			(xy 55.88 90.678) (xy 66.04 90.678)
 		)
@@
 	)
 	(symbol
+		(lib_id "Mechanical:MountingHole_Pad")
+		(at 87.63 38.1 0)
+		(unit 1)
+		(exclude_from_sim yes)
+		(in_bom no)
+		(on_board yes)
+		(dnp no)
+		(property "Reference" "H1"
+			(at 86.36 33.782 0)
+			(effects
+				(font
+					(size 1.27 1.27)
+				)
+				(justify left)
+			)
+		)
+		(property "Value" "MountingHole_Pad"
+			(at 91.186 38.0999 0)
+			(effects
+				(font
+					(size 1.27 1.27)
+				)
+				(justify left)
+				(hide yes)
+			)
+		)
+		(property "Footprint" "MountingHole:MountingHole_3.2mm_M3_ISO7380_Pad_TopBottom"
+			(at 87.63 38.1 0)
+			(effects
+				(font
+					(size 1.27 1.27)
+				)
+				(hide yes)
+			)
+		)
+		(property "Datasheet" "~"
+			(at 87.63 38.1 0)
+			(effects
+				(font
+					(size 1.27 1.27)
+				)
+				(hide yes)
+			)
+		)
+		(property "Description" "Mounting Hole with connection"
+			(at 87.63 38.1 0)
+			(effects
+				(font
+					(size 1.27 1.27)
+				)
+				(hide yes)
+			)
+		)
+		(pin "1"
+		)
+		(instances
+			(project ""
+				(path "/a200339a-72b8-45b5-a453-e4d4f113bf3a"
+					(reference "H1")
+					(unit 1)
+				)
+			)
+		)
+	)
+	(symbol
 		(lib_id "Device:R")
 		(at 160.02 86.868 0)
@@
 					(unit 1)
 				)
+			)
+		)
+	)
+	(symbol
+		(lib_id "power:GND")
+		(at 87.63 43.434 0)
+		(unit 1)
+		(exclude_from_sim no)
+		(in_bom yes)
+		(on_board yes)
+		(dnp no)
+		(fields_autoplaced yes)
+		(property "Reference" "#PWR03"
+			(at 87.63 49.784 0)
+			(effects
+				(font
+					(size 1.27 1.27)
+				)
+				(hide yes)
+			)
+		)
+		(property "Value" "GND"
+			(at 87.63 48.26 0)
+			(effects
+				(font
+					(size 1.27 1.27)
+				)
+			)
+		)
+		(property "Footprint" ""
+			(at 87.63 43.434 0)
+			(effects
+				(font
+					(size 1.27 1.27)
+				)
+				(hide yes)
+			)
+		)
+		(property "Datasheet" ""
+			(at 87.63 43.434 0)
+			(effects
+				(font
+					(size 1.27 1.27)
+				)
+				(hide yes)
+			)
+		)
+		(property "Description" "Power symbol creates a global label with name \"GND\" , ground"
+			(at 87.63 43.434 0)
+			(effects
+				(font
+					(size 1.27 1.27)
+				)
+				(hide yes)
+			)
+		)
+		(pin "1"
+		)
+		(instances
+			(project ""
+				(path "/a200339a-72b8-45b5-a453-e4d4f113bf3a"
+					(reference "#PWR03")
+					(unit 1)
+				)

Commit message: feat: updates
Parts:
- R1, R11, R13, R15, R3, R5, R7, R9: value 20000 -> 15k
- R10, R12, R14, R16, R2, R4, R6, R8: value 10000 -> 7.5k
Connections:
- net +3.3V renamed +5V
Changed lines of the file:
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@@
 	)
 	(junction
-		(at 19.05 80.518)
+		(at 17.018 80.264)
 		(diameter 0)
 		(color 0 0 0 0)
@@
 	(wire
 		(pts
-			(xy 19.05 80.518) (xy 24.765 80.518)
+			(xy 17.018 80.264) (xy 17.272 80.264)
 		)
 		(stroke
@@
 	(wire
 		(pts
+			(xy 17.272 80.264) (xy 17.272 80.518)
+		)
+		(stroke
+			(width 0)
+			(type default)
+		)
+	)
+	(wire
+		(pts
 			(xy 134.62 73.533) (xy 134.62 80.518)
 		)
@@
 	(wire
 		(pts
+			(xy 17.272 80.518) (xy 24.765 80.518)
+		)
+		(stroke
+			(width 0)
+			(type default)
+		)
+	)
+	(wire
+		(pts
 			(xy 224.79 80.518) (xy 239.395 80.518)
 		)
@@
 			)
 		)
-		(property "Value" "10000"
+		(property "Value" "7.5k"
 			(at 130.175 88.1379 0)
 			(effects
@@
 			)
 		)
-		(property "Value" "10000"
+		(property "Value" "7.5k"
 			(at 161.925 88.1379 0)
 			(effects
@@
 			)
 		)
-		(property "Value" "20000"
+		(property "Value" "15k"
 			(at 182.245 88.1379 0)
 			(effects
@@
 			)
 		)
-		(property "Value" "20000"
+		(property "Value" "15k"
 			(at 120.65 88.1379 0)
 			(effects
@@
 			)
 		)
-		(property "Value" "20000"
+		(property "Value" "15k"
 			(at 27.305 88.1379 0)
 			(effects
@@
 	)
 	(symbol
+		(lib_id "power:+5V")
+		(at 19.05 60.198 0)
+		(unit 1)
+		(exclude_from_sim no)
+		(in_bom yes)
+		(on_board yes)
+		(dnp no)
+		(fields_autoplaced yes)
+		(property "Reference" "#PWR04"
+			(at 19.05 64.008 0)
+			(effects
+				(font
+					(size 1.27 1.27)
+				)
+				(hide yes)
+			)
+		)
+		(property "Value" "+5V"
+			(at 19.05 55.118 0)
+			(effects
+				(font
+					(size 1.27 1.27)
+				)
+			)
+		)
+		(property "Footprint" ""
+			(at 19.05 60.198 0)
+			(effects
+				(font
+					(size 1.27 1.27)
+				)
+				(hide yes)
+			)
+		)
+		(property "Datasheet" ""
+			(at 19.05 60.198 0)
+			(effects
+				(font
+					(size 1.27 1.27)
+				)
+				(hide yes)
+			)
+		)
+		(property "Description" "Power symbol creates a global label with name \"+5V\""
+			(at 19.05 60.198 0)
+			(effects
+				(font
+					(size 1.27 1.27)
+				)
+				(hide yes)
+			)
+		)
+		(pin "1"
+		)
+		(instances
+			(project ""
+				(path "/a200339a-72b8-45b5-a453-e4d4f113bf3a"
+					(reference "#PWR04")
+					(unit 1)
+				)
+			)
+		)
+	)
+	(symbol
 		(lib_id "Device:R")
 		(at 239.395 86.868 0)
@@
 			)
 		)
-		(property "Value" "20000"
+		(property "Value" "15k"
 			(at 241.935 88.1379 0)
 			(effects
@@
 			)
 		)
-		(property "Value" "20000"
+		(property "Value" "15k"
 			(at 90.17 88.1379 0)
 			(effects
@@
 	(symbol
 		(lib_id "power:PWR_FLAG")
-		(at 19.05 80.518 0)
+		(at 17.018 80.264 0)
 		(unit 1)
 		(exclude_from_sim no)
@@
 		(fields_autoplaced yes)
 		(property "Reference" "#FLG02"
-			(at 19.05 78.613 0)
+			(at 17.018 78.359 0)
 			(effects
 				(font
@@
 		)
 		(property "Value" "PWR_FLAG"
-			(at 19.05 76.2 0)
+			(at 17.018 75.946 0)
 			(effects
 				(font
@@
 		)
 		(property "Footprint" ""
-			(at 19.05 80.518 0)
+			(at 17.018 80.264 0)
 			(effects
 				(font
@@
 		)
 		(property "Datasheet" "~"
-			(at 19.05 80.518 0)
+			(at 17.018 80.264 0)
 			(effects
 				(font
@@
 		)
 		(property "Description" "Special symbol for telling ERC where power comes from"
-			(at 19.05 80.518 0)
+			(at 17.018 80.264 0)
 			(effects
 				(font
@@
 			)
 		)
-		(property "Value" "10000"
+		(property "Value" "7.5k"
 			(at 221.615 88.1379 0)
 			(effects
@@
 			)
 		)
-		(property "Value" "10000"
+		(property "Value" "7.5k"
 			(at 99.695 88.1379 0)
 			(effects
@@
 			)
 		)
-		(property "Value" "10000"
+		(property "Value" "7.5k"
 			(at 36.83 88.1379 0)
 			(effects
@@
 	(symbol
 		(lib_id "power:GND")
-		(at 19.05 80.518 0)
+		(at 17.018 80.264 0)
 		(unit 1)
 		(exclude_from_sim no)
@@
 		(fields_autoplaced yes)
 		(property "Reference" "#PWR02"
-			(at 19.05 86.868 0)
+			(at 17.018 86.614 0)
 			(effects
 				(font
@@
 		)
 		(property "Value" "GND"
-			(at 19.05 85.598 0)
+			(at 17.018 85.344 0)
 			(effects
 				(font
@@
 		)
 		(property "Footprint" ""
-			(at 19.05 80.518 0)
+			(at 17.018 80.264 0)
 			(effects
 				(font
@@
 		)
 		(property "Datasheet" ""
-			(at 19.05 80.518 0)
+			(at 17.018 80.264 0)
 			(effects
 				(font
@@
 		)
 		(property "Description" "Power symbol creates a global label with name \"GND\" , ground"
-			(at 19.05 80.518 0)
+			(at 17.018 80.264 0)
 			(effects
 				(font
@@
 			)
 		)
-		(property "Value" "20000"
+		(property "Value" "15k"
 			(at 212.09 88.1379 0)
 			(effects
@@
 			)
 		)
-		(property "Value" "10000"
+		(property "Value" "7.5k"
 			(at 191.77 88.1379 0)
 			(effects
@@
 			)
 		)
-		(property "Value" "20000"
+		(property "Value" "15k"
 			(at 58.42 88.1379 0)
 			(effects
@@
 	)
 	(symbol
-		(lib_id "power:+3.3V")
-		(at 19.05 60.198 0)
-		(unit 1)
-		(exclude_from_sim no)
-		(in_bom yes)
-		(on_board yes)
-		(dnp no)
-		(fields_autoplaced yes)
-		(property "Reference" "#PWR01"
-			(at 19.05 64.008 0)
-			(effects
-				(font
-					(size 1.27 1.27)
-				)
-				(hide yes)
-			)
-		)
-		(property "Value" "+3.3V"
-			(at 19.05 55.118 0)
-			(effects
-				(font
-					(size 1.27 1.27)
-				)
-			)
-		)
-		(property "Footprint" ""
-			(at 19.05 60.198 0)
-			(effects
-				(font
-					(size 1.27 1.27)
-				)
-				(hide yes)
-			)
-		)
-		(property "Datasheet" ""
-			(at 19.05 60.198 0)
-			(effects
-				(font
-					(size 1.27 1.27)
-				)
-				(hide yes)
-			)
-		)
-		(property "Description" "Power symbol creates a global label with name \"+3.3V\""
-			(at 19.05 60.198 0)
-			(effects
-				(font
-					(size 1.27 1.27)
-				)
-				(hide yes)
-			)
-		)
-		(pin "1"
-		)
-		(instances
-			(project "MagnetronSensorArm"
-				(path "/a200339a-72b8-45b5-a453-e4d4f113bf3a"
-					(reference "#PWR01")
-					(unit 1)
-				)
-			)
-		)
-	)
-	(symbol
 		(lib_id "Device:R")
 		(at 149.86 86.868 0)
@@
 			)
 		)
-		(property "Value" "20000"
+		(property "Value" "15k"
 			(at 152.4 88.1379 0)
 			(effects
@@
 			)
 		)
-		(property "Value" "10000"
+		(property "Value" "7.5k"
 			(at 67.945 88.1379 0)
 			(effects
@@
 			)
 		)
-		(property "Value" "10000"
+		(property "Value" "7.5k"
 			(at 251.46 88.1379 0)
 			(effects
