File: hardware/kicad/MagnetronSensorArm/MagnetronSensorArm.kicad_pcb (KiCad board)
At the start: 4 copper layers, 130 x 11.4 mm, 33 parts, among them J1 Conn_02x05_Odd_Even, U1 A1301KLHLT-T, U2 A1301KLHLT-T, U3 A1301KLHLT-T, U4 A1301KLHLT-T, U5 A1301KLHLT-T, U6 A1301KLHLT-T, U7 A1301KLHLT-T, U8 A1301KLHLT-T

Commit message: feat: break into multiple boards
Routing:
- net GND: vias 16 -> 17
- added copper zone on B.Cu, net GND
- added copper zone on F.Cu, net GND
Changed lines of the file:
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@@
+	)
+	(via
+		(at 192.786 102.616)
+		(size 0.6)
+		(drill 0.3)
+		(layers "F.Cu" "B.Cu")
+		(net 2)
 	)
 	(via
@@
 	)
 	(zone
+		(net 2)
+		(net_name "GND")
+		(layer "F.Cu")
+		(hatch edge 0.5)
+		(priority 1)
+		(connect_pads
+			(clearance 0.5)
+		)
+		(min_thickness 0.25)
+		(filled_areas_thickness no)
+		(fill yes
+			(thermal_gap 0.5)
+			(thermal_bridge_width 0.5)
+		)
+		(polygon
+			(pts
+				(xy 84.074 96.774) (xy 84.074 107.696) (xy 213.614 107.696) (xy 213.614 96.774)
+			)
+		)
+	)
+	(zone
+		(net 2)
+		(net_name "GND")
+		(layer "B.Cu")
+		(hatch edge 0.5)
+		(priority 3)
+		(connect_pads
+			(clearance 0.5)
+		)
+		(min_thickness 0.25)
+		(filled_areas_thickness no)
+		(fill yes
+			(thermal_gap 0.5)
+			(thermal_bridge_width 0.5)
+		)
+		(polygon
+			(pts
+				(xy 84.074 96.774) (xy 84.074 107.696) (xy 213.614 107.696) (xy 213.614 96.774)
+			)
+		)
+	)
+	(zone

Commit message: feat: cleanup
Parts:
- added H1: MountingHole_Pad, MountingHole:MountingHole_3.2mm_M3_ISO7380_Pad_TopBottom, F.Cu at (87.1, 99.8)
Changed lines of the file:
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@@
 		)
+	)
+	(footprint "MountingHole:MountingHole_3.2mm_M3_ISO7380_Pad_TopBottom"
+		(layer "F.Cu")
+		(at 87.122 99.822)
+		(descr "Mounting Hole 3.2mm, M3, ISO7380")
+		(tags "mounting hole 3.2mm m3 iso7380")
+		(property "Reference" "H1"
+			(at 0 -3.85 0)
+			(layer "F.SilkS")
+			(hide yes)
+			(effects
+				(font
+					(size 1 1)
+					(thickness 0.15)
+				)
+			)
+		)
+		(property "Value" "MountingHole_Pad"
+			(at 0 3.85 0)
+			(layer "F.Fab")
+			(hide yes)
+			(effects
+				(font
+					(size 1 1)
+					(thickness 0.15)
+				)
+			)
+		)
+		(property "Datasheet" ""
+			(at 0 0 0)
+			(unlocked yes)
+			(layer "F.Fab")
+			(hide yes)
+			(effects
+				(font
+					(size 1.27 1.27)
+					(thickness 0.15)
+				)
+			)
+		)
+		(property "Description" "Mounting Hole with connection"
+			(at 0 0 0)
+			(unlocked yes)
+			(layer "F.Fab")
+			(hide yes)
+			(effects
+				(font
+					(size 1.27 1.27)
+					(thickness 0.15)
+				)
+			)
+		)
+		(property ki_fp_filters "MountingHole*Pad*")
+		(sheetname "/")
+		(sheetfile "MagnetronSensorArm.kicad_sch")
+		(attr exclude_from_pos_files exclude_from_bom)
+		(fp_circle
+			(center 0 0)
+			(end 2.85 0)
+			(stroke
+				(width 0.15)
+				(type solid)
+			)
+			(fill no)
+			(layer "Cmts.User")
+		)
+		(fp_circle
+			(center 0 0)
+			(end 3.1 0)
+			(stroke
+				(width 0.05)
+				(type solid)
+			)
+			(fill no)
+			(layer "F.CrtYd")
+		)
+		(fp_text user "${REFERENCE}"
+			(at 0 0 0)
+			(layer "F.Fab")
+			(effects
+				(font
+					(size 1 1)
+					(thickness 0.15)
+				)
+			)
+		)
+		(pad "1" thru_hole circle
+			(at 0 0)
+			(size 3.6 3.6)
+			(drill 3.2)
+			(layers "*.Cu" "*.Mask")
+			(remove_unused_layers no)
+			(net 2 "GND")
+			(pinfunction "1")
+			(pintype "input")
+		)
+		(pad "1" connect circle
+			(at 0 0)
+			(size 5.7 5.7)
+			(layers "F.Cu" "F.Mask")
+			(net 2 "GND")
+			(pinfunction "1")
+			(pintype "input")
+		)
+		(pad "1" connect circle
+			(at 0 0)
+			(size 5.7 5.7)
+			(layers "B.Cu" "B.Mask")
+			(net 2 "GND")
+			(pinfunction "1")
+			(pintype "input")
+		)
+		(embedded_fonts no)
 	)
 	(footprint "Package_TO_SOT_SMD:SOT-23W"

Commit message: feat: updates
Parts:
- R1, R11, R13, R15, R3, R5, R7, R9: value 20000 -> 15k
- R10, R12, R14, R16, R2, R4, R6, R8: value 10000 -> 7.5k
Connections:
- net +3.3V renamed +5V
Changed lines of the file:
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@@
 	(net 4 "/hall4")
 	(net 5 "/hall2")
-	(net 6 "+3.3V")
+	(net 6 "+5V")
 	(net 7 "/hall1")
 	(net 8 "/hall5")
@@
 			(layers "F.Cu" "F.Mask" "F.Paste")
 			(roundrect_rratio 0.25)
-			(net 6 "+3.3V")
+			(net 6 "+5V")
 			(pinfunction "VCC")
 			(pintype "power_in")
@@
 			(layers "F.Cu" "F.Mask" "F.Paste")
 			(roundrect_rratio 0.25)
-			(net 6 "+3.3V")
+			(net 6 "+5V")
 			(pinfunction "VCC")
 			(pintype "power_in")
@@
 			(layers "F.Cu" "F.Mask" "F.Paste")
 			(roundrect_rratio 0.25)
-			(net 6 "+3.3V")
+			(net 6 "+5V")
 			(pinfunction "VCC")
 			(pintype "power_in")
@@
 			(layers "F.Cu" "F.Mask" "F.Paste")
 			(roundrect_rratio 0.25)
-			(net 6 "+3.3V")
+			(net 6 "+5V")
 			(pinfunction "VCC")
 			(pintype "power_in")
@@
 			(layers "F.Cu" "F.Mask" "F.Paste")
 			(roundrect_rratio 0.25)
-			(net 6 "+3.3V")
+			(net 6 "+5V")
 			(pinfunction "VCC")
 			(pintype "power_in")
@@
 			(layers "F.Cu" "F.Mask" "F.Paste")
 			(roundrect_rratio 0.25)
-			(net 6 "+3.3V")
+			(net 6 "+5V")
 			(pinfunction "VCC")
 			(pintype "power_in")
@@
 			(layers "F.Cu" "F.Mask" "F.Paste")
 			(roundrect_rratio 0.25)
-			(net 6 "+3.3V")
+			(net 6 "+5V")
 			(pinfunction "VCC")
 			(pintype "power_in")
@@
 			(layers "F.Cu" "F.Mask" "F.Paste")
 			(roundrect_rratio 0.25)
-			(net 6 "+3.3V")
+			(net 6 "+5V")
 			(pinfunction "VCC")
 			(pintype "power_in")
@@
 			(remove_unused_layers no)
 			(roundrect_rratio 0.147059)
-			(net 6 "+3.3V")
+			(net 6 "+5V")
 			(pinfunction "Pin_1")
 			(pintype "passive")
@@
 			)
 		)
-		(property "Value" "10000"
+		(property "Value" "7.5k"
 			(at 0 -1.65 90)
 			(layer "B.Fab")
@@
 			)
 		)
-		(property "Value" "10000"
+		(property "Value" "7.5k"
 			(at 0 -1.65 90)
 			(layer "B.Fab")
@@
 			)
 		)
-		(property "Value" "20000"
+		(property "Value" "15k"
 			(at 0 -1.65 90)
 			(layer "B.Fab")
@@
 			)
 		)
-		(property "Value" "20000"
+		(property "Value" "15k"
 			(at 0 -1.65 90)
 			(layer "B.Fab")
@@
 			)
 		)
-		(property "Value" "20000"
+		(property "Value" "15k"
 			(at 0 -1.65 90)
 			(layer "B.Fab")
@@
 			)
 		)
-		(property "Value" "20000"
+		(property "Value" "15k"
 			(at 0 -1.65 90)
 			(layer "B.Fab")
@@
 			)
 		)
-		(property "Value" "20000"
+		(property "Value" "15k"
 			(at 0 -1.65 90)
 			(layer "B.Fab")
@@
 			(layers "B.Cu" "B.Mask" "B.Paste")
 			(roundrect_rratio 0.212766)
-			(net 6 "+3.3V")
+			(net 6 "+5V")
 			(pintype "passive")
 		)
@@
 			(layers "B.Cu" "B.Mask" "B.Paste")
 			(roundrect_rratio 0.212766)
-			(net 6 "+3.3V")
+			(net 6 "+5V")
 			(pintype "passive")
 		)
@@
 			)
 		)
-		(property "Value" "10000"
+		(property "Value" "7.5k"
 			(at 0 -1.65 90)
 			(layer "B.Fab")
@@
 			(layers "B.Cu" "B.Mask" "B.Paste")
 			(roundrect_rratio 0.212766)
-			(net 6 "+3.3V")
+			(net 6 "+5V")
 			(pintype "passive")
 		)
@@
 			(layers "B.Cu" "B.Mask" "B.Paste")
 			(roundrect_rratio 0.212766)
-			(net 6 "+3.3V")
+			(net 6 "+5V")
 			(pintype "passive")
 		)
@@
 			)
 		)
-		(property "Value" "10000"
+		(property "Value" "7.5k"
 			(at 0 -1.65 90)
 			(layer "B.Fab")
@@
 			)
 		)
-		(property "Value" "20000"
+		(property "Value" "15k"
 			(at 0 -1.65 90)
 			(layer "B.Fab")
@@
 			)
 		)
-		(property "Value" "10000"
+		(property "Value" "7.5k"
 			(at 0 -1.65 90)
 			(layer "B.Fab")
@@
 			(layers "B.Cu" "B.Mask" "B.Paste")
 			(roundrect_rratio 0.212766)
-			(net 6 "+3.3V")
+			(net 6 "+5V")
 			(pintype "passive")
 		)
@@
 			)
 		)
-		(property "Value" "20000"
+		(property "Value" "15k"
 			(at 0 -1.65 90)
 			(layer "B.Fab")
@@
 			(layers "B.Cu" "B.Mask" "B.Paste")
 			(roundrect_rratio 0.212766)
-			(net 6 "+3.3V")
+			(net 6 "+5V")
 			(pintype "passive")
 		)
@@
 			(layers "B.Cu" "B.Mask" "B.Paste")
 			(roundrect_rratio 0.212766)
-			(net 6 "+3.3V")
+			(net 6 "+5V")
 			(pintype "passive")
 		)
@@
 			)
 		)
-		(property "Value" "10000"
+		(property "Value" "7.5k"
 			(at 0 -1.65 90)
 			(layer "B.Fab")
@@
 			(layers "B.Cu" "B.Mask" "B.Paste")
 			(roundrect_rratio 0.212766)
-			(net 6 "+3.3V")
+			(net 6 "+5V")
 			(pintype "passive")
 		)
@@
 			)
 		)
-		(property "Value" "10000"
+		(property "Value" "7.5k"
 			(at 0 -1.65 90)
 			(layer "B.Fab")
@@
 			)
 		)
-		(property "Value" "10000"
+		(property "Value" "7.5k"
 			(at 0 -1.65 90)
 			(layer "B.Fab")
@@
 			)
 		)
-		(property "Value" "20000"
+		(property "Value" "15k"
 			(at 0 -1.65 90)
 			(layer "B.Fab")
@@
 	(zone
 		(net 6)
-		(net_name "+3.3V")
+		(net_name "+5V")
 		(layer "In2.Cu")
 		(hatch edge 0.5)

Commit message: chore: cleanup
Routing:
- net +5V: track 22.3 -> 143.8 mm
