File: hardware/kicad/MagnetronUI/encoder_breakout.kicad_sch (KiCad schematic)
At the start: 10 parts, among them SW3 RotaryEncoder_Switch_MP

Commit message: feat: cleanup
Parts:
- removed C3, C4, C5: .01uf, Capacitor_SMD:C_0805_2012Metric_Pad1.18x1.45mm_HandSolder, symbol Device:C
- removed R10, R5, R7, R9: 10k, Resistor_SMD:R_0805_2012Metric_Pad1.20x1.40mm_HandSolder, symbol Device:R
Connections:
- net encoder_a: now also R6.2, SW3.A
- net encoder_b: now also R8.1, SW3.B
- net encoder_btn: now also SW3.S2

Commit message: feat: updates
Parts:
- renumbered R6 to R1, R8 to R2, SW3 to SW2
Changed lines of the file:
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@@
 		(on_board yes)
 		(dnp no)
-		(property "Reference" "R8"
+		(property "Reference" "R2"
 			(at 108.712 109.474 90)
 			(effects
@@
 			(project "MagnetronUI"
 				(path "/a200339a-72b8-45b5-a453-e4d4f113bf3a/049b816c-78b4-46e7-959e-55d5048ed891"
-					(reference "R14")
-					(unit 1)
-				)
-				(path "/a200339a-72b8-45b5-a453-e4d4f113bf3a/1cc19acf-c923-4060-8480-daa71618b319"
-					(reference "R26")
-					(unit 1)
-				)
-				(path "/a200339a-72b8-45b5-a453-e4d4f113bf3a/29fb5d9d-1295-4995-9e43-9dca6b2abf48"
-					(reference "R32")
+					(reference "R10")
+					(unit 1)
+				)
+				(path "/a200339a-72b8-45b5-a453-e4d4f113bf3a/1cc19acf-c923-4060-8480-daa71618b319"
+					(reference "R4")
+					(unit 1)
+				)
+				(path "/a200339a-72b8-45b5-a453-e4d4f113bf3a/29fb5d9d-1295-4995-9e43-9dca6b2abf48"
+					(reference "R6")
 					(unit 1)
 				)
@@
 				)
 				(path "/a200339a-72b8-45b5-a453-e4d4f113bf3a/fe6b21e5-471b-4277-bf41-51eb9fbfa1a8"
-					(reference "R20")
+					(reference "R2")
 					(unit 1)
 				)
@@
 		(dnp no)
 		(fields_autoplaced yes)
-		(property "Reference" "#PWR012"
+		(property "Reference" "#PWR09"
 			(at 114.046 123.698 0)
 			(effects
@@
 			(project "MagnetronUI"
 				(path "/a200339a-72b8-45b5-a453-e4d4f113bf3a/049b816c-78b4-46e7-959e-55d5048ed891"
+					(reference "#PWR025")
+					(unit 1)
+				)
+				(path "/a200339a-72b8-45b5-a453-e4d4f113bf3a/1cc19acf-c923-4060-8480-daa71618b319"
+					(reference "#PWR013")
+					(unit 1)
+				)
+				(path "/a200339a-72b8-45b5-a453-e4d4f113bf3a/29fb5d9d-1295-4995-9e43-9dca6b2abf48"
 					(reference "#PWR017")
 					(unit 1)
 				)
-				(path "/a200339a-72b8-45b5-a453-e4d4f113bf3a/1cc19acf-c923-4060-8480-daa71618b319"
-					(reference "#PWR027")
-					(unit 1)
-				)
-				(path "/a200339a-72b8-45b5-a453-e4d4f113bf3a/29fb5d9d-1295-4995-9e43-9dca6b2abf48"
-					(reference "#PWR032")
-					(unit 1)
-				)
-				(path "/a200339a-72b8-45b5-a453-e4d4f113bf3a/826f9e2d-3f8d-4425-80ab-36554f164b3f"
-					(reference "#PWR012")
-					(unit 1)
-				)
-				(path "/a200339a-72b8-45b5-a453-e4d4f113bf3a/fe6b21e5-471b-4277-bf41-51eb9fbfa1a8"
-					(reference "#PWR022")
+				(path "/a200339a-72b8-45b5-a453-e4d4f113bf3a/826f9e2d-3f8d-4425-80ab-36554f164b3f"
+					(reference "#PWR021")
+					(unit 1)
+				)
+				(path "/a200339a-72b8-45b5-a453-e4d4f113bf3a/fe6b21e5-471b-4277-bf41-51eb9fbfa1a8"
+					(reference "#PWR09")
 					(unit 1)
 				)
@@
 		(dnp no)
 		(fields_autoplaced yes)
-		(property "Reference" "#PWR09"
+		(property "Reference" "#PWR06"
 			(at 94.742 114.554 0)
 			(effects
@@
 			(project "MagnetronUI"
 				(path "/a200339a-72b8-45b5-a453-e4d4f113bf3a/049b816c-78b4-46e7-959e-55d5048ed891"
+					(reference "#PWR022")
+					(unit 1)
+				)
+				(path "/a200339a-72b8-45b5-a453-e4d4f113bf3a/1cc19acf-c923-4060-8480-daa71618b319"
+					(reference "#PWR010")
+					(unit 1)
+				)
+				(path "/a200339a-72b8-45b5-a453-e4d4f113bf3a/29fb5d9d-1295-4995-9e43-9dca6b2abf48"
 					(reference "#PWR014")
 					(unit 1)
 				)
-				(path "/a200339a-72b8-45b5-a453-e4d4f113bf3a/1cc19acf-c923-4060-8480-daa71618b319"
-					(reference "#PWR024")
-					(unit 1)
-				)
-				(path "/a200339a-72b8-45b5-a453-e4d4f113bf3a/29fb5d9d-1295-4995-9e43-9dca6b2abf48"
-					(reference "#PWR029")
-					(unit 1)
-				)
-				(path "/a200339a-72b8-45b5-a453-e4d4f113bf3a/826f9e2d-3f8d-4425-80ab-36554f164b3f"
-					(reference "#PWR09")
-					(unit 1)
-				)
-				(path "/a200339a-72b8-45b5-a453-e4d4f113bf3a/fe6b21e5-471b-4277-bf41-51eb9fbfa1a8"
-					(reference "#PWR019")
+				(path "/a200339a-72b8-45b5-a453-e4d4f113bf3a/826f9e2d-3f8d-4425-80ab-36554f164b3f"
+					(reference "#PWR018")
+					(unit 1)
+				)
+				(path "/a200339a-72b8-45b5-a453-e4d4f113bf3a/fe6b21e5-471b-4277-bf41-51eb9fbfa1a8"
+					(reference "#PWR06")
 					(unit 1)
 				)
@@
 		(on_board yes)
 		(dnp no)
-		(property "Reference" "SW3"
+		(property "Reference" "SW2"
 			(at 99.568 94.234 0)
 			(effects
@@
 			(project "MagnetronUI"
 				(path "/a200339a-72b8-45b5-a453-e4d4f113bf3a/049b816c-78b4-46e7-959e-55d5048ed891"
+					(reference "SW6")
+					(unit 1)
+				)
+				(path "/a200339a-72b8-45b5-a453-e4d4f113bf3a/1cc19acf-c923-4060-8480-daa71618b319"
+					(reference "SW3")
+					(unit 1)
+				)
+				(path "/a200339a-72b8-45b5-a453-e4d4f113bf3a/29fb5d9d-1295-4995-9e43-9dca6b2abf48"
 					(reference "SW4")
 					(unit 1)
 				)
-				(path "/a200339a-72b8-45b5-a453-e4d4f113bf3a/1cc19acf-c923-4060-8480-daa71618b319"
-					(reference "SW6")
-					(unit 1)
-				)
-				(path "/a200339a-72b8-45b5-a453-e4d4f113bf3a/29fb5d9d-1295-4995-9e43-9dca6b2abf48"
-					(reference "SW7")
-					(unit 1)
-				)
-				(path "/a200339a-72b8-45b5-a453-e4d4f113bf3a/826f9e2d-3f8d-4425-80ab-36554f164b3f"
-					(reference "SW3")
-					(unit 1)
-				)
-				(path "/a200339a-72b8-45b5-a453-e4d4f113bf3a/fe6b21e5-471b-4277-bf41-51eb9fbfa1a8"
+				(path "/a200339a-72b8-45b5-a453-e4d4f113bf3a/826f9e2d-3f8d-4425-80ab-36554f164b3f"
 					(reference "SW5")
+					(unit 1)
+				)
+				(path "/a200339a-72b8-45b5-a453-e4d4f113bf3a/fe6b21e5-471b-4277-bf41-51eb9fbfa1a8"
+					(reference "SW2")
 					(unit 1)
 				)
@@
 		(dnp no)
 		(fields_autoplaced yes)
-		(property "Reference" "#PWR011"
+		(property "Reference" "#PWR08"
 			(at 120.142 94.234 0)
 			(effects
@@
 			(project "MagnetronUI"
 				(path "/a200339a-72b8-45b5-a453-e4d4f113bf3a/049b816c-78b4-46e7-959e-55d5048ed891"
+					(reference "#PWR024")
+					(unit 1)
+				)
+				(path "/a200339a-72b8-45b5-a453-e4d4f113bf3a/1cc19acf-c923-4060-8480-daa71618b319"
+					(reference "#PWR012")
+					(unit 1)
+				)
+				(path "/a200339a-72b8-45b5-a453-e4d4f113bf3a/29fb5d9d-1295-4995-9e43-9dca6b2abf48"
 					(reference "#PWR016")
 					(unit 1)
 				)
-				(path "/a200339a-72b8-45b5-a453-e4d4f113bf3a/1cc19acf-c923-4060-8480-daa71618b319"
-					(reference "#PWR026")
-					(unit 1)
-				)
-				(path "/a200339a-72b8-45b5-a453-e4d4f113bf3a/29fb5d9d-1295-4995-9e43-9dca6b2abf48"
-					(reference "#PWR031")
-					(unit 1)
-				)
-				(path "/a200339a-72b8-45b5-a453-e4d4f113bf3a/826f9e2d-3f8d-4425-80ab-36554f164b3f"
-					(reference "#PWR011")
-					(unit 1)
-				)
-				(path "/a200339a-72b8-45b5-a453-e4d4f113bf3a/fe6b21e5-471b-4277-bf41-51eb9fbfa1a8"
-					(reference "#PWR021")
+				(path "/a200339a-72b8-45b5-a453-e4d4f113bf3a/826f9e2d-3f8d-4425-80ab-36554f164b3f"
+					(reference "#PWR020")
+					(unit 1)
+				)
+				(path "/a200339a-72b8-45b5-a453-e4d4f113bf3a/fe6b21e5-471b-4277-bf41-51eb9fbfa1a8"
+					(reference "#PWR08")
 					(unit 1)
 				)
@@
 		(on_board yes)
 		(dnp no)
-		(property "Reference" "R6"
+		(property "Reference" "R1"
 			(at 103.632 109.474 90)
 			(effects
@@
 			(project "MagnetronUI"
 				(path "/a200339a-72b8-45b5-a453-e4d4f113bf3a/049b816c-78b4-46e7-959e-55d5048ed891"
-					(reference "R12")
-					(unit 1)
-				)
-				(path "/a200339a-72b8-45b5-a453-e4d4f113bf3a/1cc19acf-c923-4060-8480-daa71618b319"
-					(reference "R24")
-					(unit 1)
-				)
-				(path "/a200339a-72b8-45b5-a453-e4d4f113bf3a/29fb5d9d-1295-4995-9e43-9dca6b2abf48"
-					(reference "R30")
-					(unit 1)
-				)
-				(path "/a200339a-72b8-45b5-a453-e4d4f113bf3a/826f9e2d-3f8d-4425-80ab-36554f164b3f"
-					(reference "R6")
-					(unit 1)
-				)
-				(path "/a200339a-72b8-45b5-a453-e4d4f113bf3a/fe6b21e5-471b-4277-bf41-51eb9fbfa1a8"
-					(reference "R18")
+					(reference "R9")
+					(unit 1)
+				)
+				(path "/a200339a-72b8-45b5-a453-e4d4f113bf3a/1cc19acf-c923-4060-8480-daa71618b319"
+					(reference "R3")
+					(unit 1)
+				)
+				(path "/a200339a-72b8-45b5-a453-e4d4f113bf3a/29fb5d9d-1295-4995-9e43-9dca6b2abf48"
+					(reference "R5")
+					(unit 1)
+				)
+				(path "/a200339a-72b8-45b5-a453-e4d4f113bf3a/826f9e2d-3f8d-4425-80ab-36554f164b3f"
+					(reference "R7")
+					(unit 1)
+				)
+				(path "/a200339a-72b8-45b5-a453-e4d4f113bf3a/fe6b21e5-471b-4277-bf41-51eb9fbfa1a8"
+					(reference "R1")
 					(unit 1)
 				)
@@
 		(dnp no)
 		(fields_autoplaced yes)
-		(property "Reference" "#PWR010"
+		(property "Reference" "#PWR07"
 			(at 93.218 84.074 0)
 			(effects
@@
 			(project "MagnetronUI"
 				(path "/a200339a-72b8-45b5-a453-e4d4f113bf3a/049b816c-78b4-46e7-959e-55d5048ed891"
+					(reference "#PWR023")
+					(unit 1)
+				)
+				(path "/a200339a-72b8-45b5-a453-e4d4f113bf3a/1cc19acf-c923-4060-8480-daa71618b319"
+					(reference "#PWR011")
+					(unit 1)
+				)
+				(path "/a200339a-72b8-45b5-a453-e4d4f113bf3a/29fb5d9d-1295-4995-9e43-9dca6b2abf48"
 					(reference "#PWR015")
 					(unit 1)
 				)
-				(path "/a200339a-72b8-45b5-a453-e4d4f113bf3a/1cc19acf-c923-4060-8480-daa71618b319"
-					(reference "#PWR025")
-					(unit 1)
-				)
-				(path "/a200339a-72b8-45b5-a453-e4d4f113bf3a/29fb5d9d-1295-4995-9e43-9dca6b2abf48"
-					(reference "#PWR030")
-					(unit 1)
-				)
-				(path "/a200339a-72b8-45b5-a453-e4d4f113bf3a/826f9e2d-3f8d-4425-80ab-36554f164b3f"
-					(reference "#PWR010")
-					(unit 1)
-				)
-				(path "/a200339a-72b8-45b5-a453-e4d4f113bf3a/fe6b21e5-471b-4277-bf41-51eb9fbfa1a8"
-					(reference "#PWR020")
-					(unit 1)
-				)
+				(path "/a200339a-72b8-45b5-a453-e4d4f113bf3a/826f9e2d-3f8d-4425-80ab-36554f164b3f"
+					(reference "#PWR019")
+					(unit 1)
+				)
+				(path "/a200339a-72b8-45b5-a453-e4d4f113bf3a/fe6b21e5-471b-4277-bf41-51eb9fbfa1a8"
+					(reference "#PWR07")
+					(unit 1)
+				)
