File: hardware/kicad/MagetroneController/MagetroneController.kicad_pcb (KiCad board)
At the start: 4 copper layers, 80 x 80 mm, 24 parts, among them J1 Conn_01x04, J2 DIN-5_180degree, J3 DIN-5_180degree, J4 Barrel_Jack_MountingPin, J7 Conn_02x05_Odd_Even, J8 Conn_02x13_Counter_Clockwise, SW9 SW_SPST 24V, U10 Teensy4.1, U12 6N137

Commit message: chore: rename project files
Parts:
- moved H4 0.62 mm to (125.8, 138.5)
- moved H2 0.61 mm to (125.8, 68.5)
- moved H3 0.61 mm to (55.8, 138.5)
- moved H1 0.61 mm to (55.8, 68.5)
Changed lines of the file:
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@@
 	(footprint "MountingHole:MountingHole_3.2mm_M3_ISO7380_Pad_TopBottom"
 		(layer "F.Cu")
-		(at 126.238 138.938)
+		(at 125.8 138.5)
 		(descr "Mounting Hole 3.2mm, M3, ISO7380")
 		(tags "mounting hole 3.2mm m3 iso7380")
@@
 	(footprint "MountingHole:MountingHole_3.2mm_M3_ISO7380_Pad_TopBottom"
 		(layer "F.Cu")
-		(at 55.372 138.938)
+		(at 55.8 138.5)
 		(descr "Mounting Hole 3.2mm, M3, ISO7380")
 		(tags "mounting hole 3.2mm m3 iso7380")
@@
 	(footprint "MountingHole:MountingHole_3.2mm_M3_ISO7380_Pad_TopBottom"
 		(layer "F.Cu")
-		(at 126.238 68.072)
+		(at 125.8 68.5)
 		(descr "Mounting Hole 3.2mm, M3, ISO7380")
 		(tags "mounting hole 3.2mm m3 iso7380")
@@
 	(footprint "MountingHole:MountingHole_3.2mm_M3_ISO7380_Pad_TopBottom"
 		(layer "F.Cu")
-		(at 55.372 68.072)
+		(at 55.8 68.5)
 		(descr "Mounting Hole 3.2mm, M3, ISO7380")
 		(tags "mounting hole 3.2mm m3 iso7380")
@@
 		)
 	)
+	(group ""
+		(members "2e2fb419-b594-4ca8-a713-6cdc0553b79e" "35a5f1d5-bd76-48df-9876-392c817a58e8"
+			"462b7693-8eef-4b5e-9923-b5468e4fb07a" "bf45f88f-4af5-4164-a32b-c1ba331ba807"
+		)
+	)
