File: hardware/kicad/MagnetroneController/MagnetroneController.kicad_pcb (KiCad board)
At the start: 4 copper layers, 80 x 80 mm, 26 parts, among them J1 Conn_01x04, J2 DIN-5_180degree, J3 DIN-5_180degree, J4 Barrel_Jack_MountingPin, J7 Conn_02x05_Odd_Even, J8 Conn_02x13_Counter_Clockwise, SW9 SW_SPST 24V, U1 TMC2209_BTT_V1.3, U10 Teensy4.1, U12 6N137

Commit message: updates, and added tests
Routing:
- net GND: vias 20 -> 23
Changed lines of the file:
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@@
+	)
+	(via
+		(at 66.548 117.856)
+		(size 0.6)
+		(drill 0.3)
+		(layers "F.Cu" "B.Cu")
+		(net 2)
 	)
 	(via
@@
 	)
 	(via
+		(at 95.25 116.84)
+		(size 0.6)
+		(drill 0.3)
+		(layers "F.Cu" "B.Cu")
+		(net 2)
+	)
+	(via
 		(at 92.456 130.81)
 		(size 0.6)
@@
 		(size 0.6)
 		(drill 0.3)
+		(layers "F.Cu" "B.Cu")
+		(net 2)
+	)
+	(via
+		(at 84.582 89.916)
+		(size 0.6)
+		(drill 0.3)
