File: hardware/kicad/MagnetroneUI/MagnetroneUI.kicad_pcb (KiCad board)
At the start: 2 copper layers, 120 x 50 mm, 25 parts, among them J1 Conn_01x04, J2 Conn_02x13_Counter_Clockwise, Q1 BSS138, Q2 BSS138, SW1 SW_Push, SW2 RotaryEncoder_Switch_MP, SW3 RotaryEncoder_Switch_MP, SW4 RotaryEncoder_Switch_MP, SW5 RotaryEncoder_Switch_MP

Commit message: Record Designer template fixes and docs (magnet colors, platter direction, hosted link); test sketches, fabrication outputs, scripts
Other:
- board text removed: "aux2 encoder"
Changed lines of the file:
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@@
-		)
-	)
-	(gr_text "aux2 encoder"
-		(at 130.302 124.206 0)
-		(layer "F.SilkS")
-		(effects
-			(font
-				(size 1 1)
-				(thickness 0.15)
-			)
 		)
 	)
